Commit message: add camera support 3D model

File: gen3_lite_description/urdf/camera/_d435.urdf.xacro (robot description, xacro)
@@ -76,5 +76,5 @@
         </xacro:if>
         <xacro:unless value="${use_mesh}">
-          <origin xyz="0 ${-d435_cam_depth_py} 0" rpy="0 0 0" />
+          <origin xyz="-0.008 ${-d435_cam_depth_py} 0" rpy="0 0 0" />
           <geometry>
             <box size="${d435_cam_depth} ${d435_cam_width} ${d435_cam_height}" />
@@ -84,5 +84,5 @@
       </visual>
       <collision>
-        <origin xyz="0 ${-d435_cam_depth_py} 0" rpy="0 0 0" />
+        <origin xyz="-0.008 ${-d435_cam_depth_py} 0" rpy="0 0 0" />
         <geometry>
           <box size="${d435_cam_depth} ${d435_cam_width} ${d435_cam_height}" />

File: gen3_lite_description/urdf/gen3_lite.urdf.xacro (robot description, xacro)
@@ -1,6 +1,7 @@
 <?xml version="1.0"?>
-<robot name="gen3_lite" xmlns:xacro="http://ros.org/wiki/xacro">
+<robot name="$(arg name)" xmlns:xacro="http://ros.org/wiki/xacro">
     <!-- Arguments -->
-    <xacro:arg name="sim_gazebo" default="false" />
+    <xacro:arg name="name" default="gen3_lite"/>
+    <xacro:arg name="sim_gazebo" default="true" />
     <xacro:arg name="use_camera" default="false" />
     <xacro:arg name="prefix" default=""/>

File: gen3_lite_description/urdf/gen3_lite_macro.urdf.xacro (robot description, xacro)
@@ -216,7 +216,18 @@
         <!-- Optional components -->
         <xacro:if value="${use_camera}">
+            <xacro:include filename="$(find gen3_lite_description)/urdf/camera/support.urdf.xacro" />
+            <xacro:camera_inferior_support parent="dummy_link" prefix="${prefix}">
+                <origin rpy="0.0 0.0 ${M_PI/2}" xyz="0.0 0.0 0.018" />
+            </xacro:camera_inferior_support>
+            <xacro:camera_superior_support parent="dummy_link" prefix="${prefix}">
+                <origin rpy="0.0 0.0 -${M_PI/2}" xyz="0.0 0.0 0.018" />
+            </xacro:camera_superior_support>
+            <!-- <xacro:include filename="$(find gen3_lite_description)/urdf/camera/_d435.urdf.xacro" />
+            <xacro:sensor_d435 parent="dummy_link" prefix="${prefix}" name="camera_1" add_plug="false">
+                <origin rpy="${M_PI} -${M_PI/2} 0.0" xyz="0.045 0.0 0.018" />
+            </xacro:sensor_d435> -->
             <xacro:include filename="$(find gen3_lite_description)/urdf/camera/_d435.urdf.xacro" />
-            <xacro:sensor_d435 parent="dummy_link" prefix="${prefix}" name="camera_1">
-                <origin rpy="${M_PI} -${M_PI/2} 0.0" xyz="0.045 0.0 0.015" />
+            <xacro:sensor_d435 parent="camera_support_cylinder_link" prefix="${prefix}" name="camera_1" add_plug="false">
+                <origin rpy="0.0 -${M_PI/2} -${M_PI/2}" xyz="0.0 0.010 0.0" />
             </xacro:sensor_d435>
         </xacro:if>

File: gen3_lite_description/urdf/macros.urdf.xacro (robot description, xacro)
@@ -7,4 +7,7 @@
     <material name="gen3_lite_white">
         <color rgba="0.803 0.824 0.820 1" />
+    </material>
+    <material name="camera_support_dark_gray">
+        <color rgba="0.25 0.25 0.25 1"/>
     </material>
     <xacro:property name="joint_limits_config" value="${xacro.load_yaml('$(arg joint_limits)')}" />

Commit message: fix camera position

File: gen3_lite_description/urdf/camera/_d435.urdf.xacro (robot description, xacro)
@@ -29,5 +29,5 @@
       prefix
       use_mesh:=true
-      use_nominal_extrinsics:=false">
+      use_nominal_extrinsics:=true">
     <!-- The following values are approximate, and the camera node
      publishing TF values with actual calibrated camera extrinsic values -->

File: gen3_lite_description/urdf/camera/support.urdf.xacro (robot description, xacro)
@@ -51,5 +51,5 @@
     </link>
     <joint name="${prefix}camera_support_cylinder_joint" type="fixed">
-      <origin rpy="0.0 0.0 0.0" xyz="0.0 0.0575 0.0" />
+      <origin rpy="0.0 0.0 0.0" xyz="0.0 0.0625 0.0" />
       <parent link="${prefix}camera_support_superior_link" />
       <child link="${prefix}camera_support_cylinder_link" />
@@ -59,5 +59,5 @@
         <origin xyz="0.0 0 0.0" rpy="-${M_PI/2} 0 0" />
         <geometry>
-          <cylinder radius="0.009" length="0.02" />
+          <cylinder radius="0.01156" length="0.0398" />
         </geometry>
         <material name="camera_support_dark_gray" />
@@ -66,5 +66,5 @@
         <origin xyz="0.0 0 0.0" rpy="-${M_PI/2} 0 0" />
         <geometry>
-          <cylinder radius="0.009" length="0.02" />
+          <cylinder radius="0.01156" length="0.0398" />
         </geometry>
       </collision>

File: gen3_lite_description/urdf/gen3_lite_macro.urdf.xacro (robot description, xacro)
@@ -218,8 +218,8 @@
             <xacro:include filename="$(find gen3_lite_description)/urdf/camera/support.urdf.xacro" />
             <xacro:camera_inferior_support parent="dummy_link" prefix="${prefix}">
-                <origin rpy="0.0 0.0 ${M_PI/2}" xyz="0.0 0.0 0.018" />
+                <origin rpy="0.0 0.0 ${M_PI/2}" xyz="0.0 0.0 0.0133" />
             </xacro:camera_inferior_support>
             <xacro:camera_superior_support parent="dummy_link" prefix="${prefix}">
-                <origin rpy="0.0 0.0 -${M_PI/2}" xyz="0.0 0.0 0.018" />
+                <origin rpy="0.0 0.0 -${M_PI/2}" xyz="0.0 0.0 0.0133" />
             </xacro:camera_superior_support>
             <!-- <xacro:include filename="$(find gen3_lite_description)/urdf/camera/_d435.urdf.xacro" />
@@ -229,5 +229,5 @@
             <xacro:include filename="$(find gen3_lite_description)/urdf/camera/_d435.urdf.xacro" />
             <xacro:sensor_d435 parent="camera_support_cylinder_link" prefix="${prefix}" name="camera_1" add_plug="false">
-                <origin rpy="0.0 -${M_PI/2} -${M_PI/2}" xyz="0.0 0.010 0.0" />
+                <origin rpy="0.0 -${M_PI/2} -${M_PI/2}" xyz="0.0 0.0190 0.0" />
             </xacro:sensor_d435>
         </xacro:if>

File: gen3_lite_description/urdf/ros2_control/gen3_lite_ros2_control.xacro (robot description, xacro)
@@ -95,7 +95,5 @@
                 <joint name="${prefix}right_finger_bottom_joint">
                     <command_interface name="position" />
-                    <state_interface name="position">
-                        <param name="initial_value">${right_finger_bottom_joint_initial}</param>
-                    </state_interface>
+                    <state_interface name="position" />
                     <state_interface name="velocity" />
                 </joint>
