Commit message: update camera base 3D

File: gen3_lite_description/urdf/camera/support.urdf.xacro (robot description, xacro)
@@ -39,5 +39,5 @@
         <origin xyz="-0.064 0 -0.0125" rpy="0 0 0" />
         <geometry>
-          <mesh filename="package://gen3_lite_description/meshes/d435/anel_jackal_superior.STL" scale="0.001 0.001 0.001" />
+          <mesh filename="package://gen3_lite_description/meshes/d435/anel_jackal_superior_2.STL" scale="0.001 0.001 0.001" />
         </geometry>
         <material name="camera_support_dark_gray" />
@@ -46,9 +46,9 @@
         <origin xyz="-0.064 0 -0.0125" rpy="0 0 0" />
         <geometry>
-          <mesh filename="package://gen3_lite_description/meshes/d435/anel_jackal_superior.STL" scale="0.001 0.001 0.001" />
+          <mesh filename="package://gen3_lite_description/meshes/d435/anel_jackal_superior_2.STL" scale="0.001 0.001 0.001" />
         </geometry>
       </collision>
     </link>
-    <joint name="${prefix}camera_support_cylinder_joint" type="fixed">
+    <!-- <joint name="${prefix}camera_support_cylinder_joint" type="fixed">
       <origin rpy="0.0 0.0 0.0" xyz="0.0 0.0625 0.0" />
       <parent link="${prefix}camera_support_superior_link" />
@@ -69,5 +69,5 @@
         </geometry>
       </collision>
-    </link>
+    </link> -->
   </xacro:macro>
 </robot>

File: gen3_lite_description/urdf/gen3_lite_macro.urdf.xacro (robot description, xacro)
@@ -228,6 +228,6 @@
             </xacro:sensor_d435> -->
             <xacro:include filename="$(find gen3_lite_description)/urdf/camera/_d435.urdf.xacro" />
-            <xacro:sensor_d435 parent="camera_support_cylinder_link" prefix="${prefix}" name="camera_1" add_plug="false">
-                <origin rpy="0.0 -${M_PI/2} -${M_PI/2}" xyz="0.0 0.0190 0.0" />
+            <xacro:sensor_d435 parent="camera_support_superior_link" prefix="${prefix}" name="camera_1">
+                <origin rpy="0.0 -${M_PI/2} -${M_PI/2}" xyz="0.0 0.0815 0.0051" />
             </xacro:sensor_d435>
         </xacro:if>
